File: eagle/m5stack-2sided-pinheader.brd (EAGLE design)
At the start: 50 x 50 mm, 2 parts

Commit message: pcb update
Parts:
- removed PINH-FEMAIL, PINH-MAIL: 2X15, m5stack:SMD-PINH-2X15-C
- added PINH-FEMALE, PINH-MALE: M5STACK-PINHHANDSOLDER, kenu-m5stack:PINH-2X15-SMD_HANDSOLDER
Connections:
- net 3.3V: now also PINH-FEMALE.12, PINH-MALE.11; no longer PINH-FEMAIL.12, PINH-MAIL.11
- net 5V: now also PINH-FEMALE.28, PINH-MALE.27; no longer PINH-FEMAIL.28, PINH-MAIL.27
- net BATT: now also PINH-FEMALE.30, PINH-MALE.29; no longer PINH-FEMAIL.30, PINH-MAIL.29
- net G2: now also PINH-FEMALE.19, PINH-MALE.20; no longer PINH-FEMAIL.19, PINH-MAIL.20
- net G25: now also PINH-FEMALE.8, PINH-MALE.7; no longer PINH-FEMAIL.8, PINH-MAIL.7
- net G26: now also PINH-FEMALE.10, PINH-MALE.9; no longer PINH-FEMAIL.10, PINH-MAIL.9
- net G35: now also PINH-FEMALE.2, PINH-MALE.1; no longer PINH-FEMAIL.2, PINH-MAIL.1
- net G36: now also PINH-FEMALE.4, PINH-MALE.3; no longer PINH-FEMAIL.4, PINH-MAIL.3
- net G5: now also PINH-FEMALE.20, PINH-MALE.19; no longer PINH-FEMAIL.20, PINH-MAIL.19
- net GND: now also PINH-FEMALE.1, PINH-FEMALE.3, PINH-FEMALE.5, PINH-MALE.2, PINH-MALE.4, PINH-MALE.6; no longer PINH-FEMAIL.1, PINH-FEMAIL.3, PINH-FEMAIL.5, PINH-MAIL.2, PINH-MAIL.4, PINH-MAIL.6
- net HPWR: now also PINH-FEMALE.25, PINH-FEMALE.27, PINH-FEMALE.29, PINH-MALE.26, PINH-MALE.28, PINH-MALE.30; no longer PINH-FEMAIL.25, PINH-FEMAIL.27, PINH-FEMAIL.29, PINH-MAIL.26, PINH-MAIL.28, PINH-MAIL.30
- net IISIN: now also PINH-FEMALE.26, PINH-MALE.25; no longer PINH-FEMAIL.26, PINH-MAIL.25
- net IISMK: now also PINH-FEMALE.24, PINH-MALE.23; no longer PINH-FEMAIL.24, PINH-MAIL.23
- net IISOUT: now also PINH-FEMALE.23, PINH-MALE.24; no longer PINH-FEMAIL.23, PINH-MAIL.24
- net IISSK: now also PINH-FEMALE.21, PINH-MALE.22; no longer PINH-FEMAIL.21, PINH-MAIL.22
- net IISWS: now also PINH-FEMALE.22, PINH-MALE.21; no longer PINH-FEMAIL.22, PINH-MAIL.21
- net MISO: now also PINH-FEMALE.9, PINH-MALE.10; no longer PINH-FEMAIL.9, PINH-MAIL.10
- net MOSI: now also PINH-FEMALE.7, PINH-MALE.8; no longer PINH-FEMAIL.7, PINH-MAIL.8
- net RST: now also PINH-FEMALE.6, PINH-MALE.5; no longer PINH-FEMAIL.6, PINH-MAIL.5
- net RXD0: now also PINH-FEMALE.13, PINH-MALE.14; no longer PINH-FEMAIL.13, PINH-MAIL.14
- net RXD2: now also PINH-FEMALE.15, PINH-MALE.16; no longer PINH-FEMAIL.15, PINH-MAIL.16
- net SCK: now also PINH-FEMALE.11, PINH-MALE.12; no longer PINH-FEMAIL.11, PINH-MAIL.12
- net SCL: now also PINH-FEMALE.18, PINH-MALE.17; no longer PINH-FEMAIL.18, PINH-MAIL.17
- net SDA: now also PINH-FEMALE.17, PINH-MALE.18; no longer PINH-FEMAIL.17, PINH-MAIL.18
- net TXD0: now also PINH-FEMALE.14, PINH-MALE.13; no longer PINH-FEMAIL.14, PINH-MAIL.13
- net TXD2: now also PINH-FEMALE.16, PINH-MALE.15; no longer PINH-FEMAIL.16, PINH-MAIL.15
Routing:
- net GND: track 19.2 -> 18.6 mm
Other:
- outline, holes or cut-outs redrawn
- board text added: "0"
- board text added: "12"
- board text added: "13"
- board text added: "15"
- board text added: "19"
- board text added: "2"
- board text added: "23"
- board text added: "25"
- board text added: "26"
- board text added: "3.3V"
- board text added: "34"
- board text added: "35"
- board text added: "36"
- board text added: "5"
- board text added: "5V"
- board text added: "BAT"
- board text added: "GND"
- board text added: "HPWR"
- board text added: "RST"
- board text added: "RX0"
- board text added: "RX2"
- board text added: "SCK"
- board text added: "SCL"
- board text added: "SDA"
- board text added: "TX0"
- board text added: "TX2"
